File: PW-Display.kicad_sch (KiCad schematic)
At the start: 6 parts, among them U1 WeMos_D1_mini_GPIO

Commit message: Updated kicad
Connections:
- net at SOLAR.1 (CLK): now also U1.14 (D1/GPIO5); no longer U1.13 (D2/GPIO4)
- net at SOLAR.2 (DIO): now also U1.13 (D2/GPIO4); no longer U1.14 (D1/GPIO5)
Changed lines of the file:
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@@
+    (stroke (width 0) (type default) (color 0 0 0 0))
+  )
+  (wire (pts (xy 86.36 57.15) (xy 90.17 57.15))
     (stroke (width 0) (type default) (color 0 0 0 0))
   )
@@
     (stroke (width 0) (type default) (color 0 0 0 0))
   )
-  (wire (pts (xy 92.71 57.15) (xy 92.71 36.83))
+  (wire (pts (xy 92.71 36.83) (xy 92.71 60.96))
     (stroke (width 0) (type default) (color 0 0 0 0))
   )
@@
     (stroke (width 0) (type default) (color 0 0 0 0))
   )
+  (wire (pts (xy 90.17 34.29) (xy 90.17 57.15))
+    (stroke (width 0) (type default) (color 0 0 0 0))
+  )
   (wire (pts (xy 110.49 71.12) (xy 113.03 71.12))
     (stroke (width 0) (type default) (color 0 0 0 0))
@@
     (stroke (width 0) (type default) (color 0 0 0 0))
   )
+  (wire (pts (xy 86.36 60.96) (xy 92.71 60.96))
+    (stroke (width 0) (type default) (color 0 0 0 0))
+  )
   (wire (pts (xy 105.41 73.66) (xy 105.41 72.39))
     (stroke (width 0) (type default) (color 0 0 0 0))
@@
     (stroke (width 0) (type default) (color 0 0 0 0))
   )
-  (wire (pts (xy 113.03 34.29) (xy 91.44 34.29))
+  (wire (pts (xy 90.17 34.29) (xy 113.03 34.29))
     (stroke (width 0) (type default) (color 0 0 0 0))
   )
@@
     (stroke (width 0) (type default) (color 0 0 0 0))
   )
-  (wire (pts (xy 86.36 60.96) (xy 91.44 60.96))
-    (stroke (width 0) (type default) (color 0 0 0 0))
-  )
   (wire (pts (xy 113.03 68.58) (xy 107.95 68.58))
-    (stroke (width 0) (type default) (color 0 0 0 0))
-  )
-  (wire (pts (xy 86.36 57.15) (xy 92.71 57.15))
     (stroke (width 0) (type default) (color 0 0 0 0))
   )
@@
     (stroke (width 0) (type default) (color 0 0 0 0))
   )
-  (wire (pts (xy 91.44 34.29) (xy 91.44 60.96))
-    (stroke (width 0) (type default) (color 0 0 0 0))
-  )
